File: hardware/KiCad/mini-MCU-LINK-Integrated/mini-MCU-LINK-Integrated.kicad_pcb (KiCad board)
At the start: 2 copper layers, 57 parts, among them J1 USB4110-GF-A_REVB, J2 BM03B-SRSS-TB, J3 Conn_02x05_Odd_Even, Q1 PMDXB290UNE, Q2 PMDXB290UNE, Q3 PMDXB290UNE, Q4 PMDXB290UNE, SW1 KMR221GLFS, U1 XC6227C331PR-G, U2 LPC55S69JBD64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

Commit message: Remove extraneous PMEG3005AESFYL whitespace/newline
Parts:
- D3: value PMEG3005AESFYL -> PMEG3005AESFYL
Changed lines of the file:
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@@
         (effects (font (size 0.8 0.8) (thickness 0.15)))
     )
-    (fp_text value "PMEG3005AESFYL\n" (at 0 1.05) (layer "F.Fab")
+    (fp_text value "PMEG3005AESFYL" (at 0 1.05) (layer "F.Fab")
         (effects (font (size 1 1) (thickness 0.15)))
     )
