File: hardware/KiCad/mini-MCU-LINK-Standalone/MCU-Link-Standalone.kicad_pcb (KiCad board)
At the start: 2 copper layers, 46 x 19 mm, 69 parts, among them J1 USB4110-GF-A_REVB, J2 BM03B-SRSS-TB, J3 Conn_02x05_Odd_Even, Q1 PMDXB290UNE, Q2 PMDXB290UNE, Q3 PMDXB290UNE, SW1 KMR221GLFS, U1 XC6227C331PR-G, U2 LPC55S69JBD64, U3 STMPS2141STR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

Commit message: Remove extraneous PMEG3005AESFYL whitespace/newline
Parts:
- D4: value PMEG3005AESFYL -> PMEG3005AESFYL
Changed lines of the file:
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@@
 			)
 		)
-		(property "Value" "PMEG3005AESFYL\n"
+		(property "Value" "PMEG3005AESFYL"
 			(at 0 1.05 0)
 			(unlocked yes)
