File: hardware/KiCad/mini-MCU-LINK-Standalone/mculink_standalone_debug_uart.kicad_sch (KiCad schematic)
At the start: 26 parts, among them J2 BM03B-SRSS-TB, J3 Conn_02x05_Odd_Even, Q1 PMDXB290UNE, Q2 PMDXB290UNE, Q3 PMDXB290UNE, SW1 KMR221GLFS, U2 LPC55S69JBD64, U3 STMPS2141STR

Commit message: Remove extraneous PMEG3005AESFYL whitespace/newline
Parts:
- D4: value PMEG3005AESFYL -> PMEG3005AESFYL
Changed lines of the file:
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@@
 			)
 		)
-		(property "Value" "PMEG3005AESFYL\n"
+		(property "Value" "PMEG3005AESFYL"
 			(at 154.94 168.91 0)
 			(effects
